File: particle_detector/Breakout/Comparator Breakout MAX9031.brd (EAGLE design)
At the start: 23 x 18 mm, 3 parts

Commit message: revised boards from a while ago
Routing:
- net V-: track 17.4 -> 18.7 mm
- net GND: track 26.6 -> 27.8 mm
Changed lines of the file:
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@@
 <contactref element="U$1" pad="5"/>
 <contactref element="JP1" pad="4"/>
-<wire x1="7.3" y1="7.05" x2="7.28" y2="7.03" width="0.1524" layer="1"/>
+<wire x1="7.3" y1="7.05" x2="7.28" y2="6.98" width="0.1524" layer="1"/>
 <wire x1="7.3" y1="13.78" x2="7.3" y2="7.05" width="0.4064" layer="1"/>
 <wire x1="7.3" y1="7.05" x2="7.2848" y2="7.0348" width="0.4064" layer="1"/>
@@
 <wire x1="6.2476" y1="14.69668125" x2="8.06091875" y2="16.51" width="0.4064" layer="1"/>
 <wire x1="8.06091875" y1="16.51" x2="21.59" y2="16.51" width="0.4064" layer="1"/>
-<wire x1="5.31" y1="10.31" x2="4" y2="9" width="0.4064" layer="1"/>
-<wire x1="5.31" y1="10.31" x2="5.31" y2="13.69" width="0.4064" layer="1"/>
-<wire x1="4" y1="6.4" x2="4.7873625" y2="6.4" width="0.4064" layer="1"/>
-<wire x1="4.7873625" y1="6.4" x2="4.8073625" y2="6.38" width="0.4064" layer="1"/>
-<wire x1="4" y1="9" x2="4" y2="6.4" width="0.4064" layer="1"/>
-<wire x1="4.8073625" y1="6.38" x2="5.08" y2="6.38" width="0" layer="19" extent="1-1"/>
+<wire x1="5.08" y1="6.03" x2="4.03" y2="6.03" width="0.5" layer="1"/>
+<wire x1="4.03" y1="6.03" x2="4" y2="6" width="0.5" layer="1"/>
+<wire x1="4" y1="6" x2="4" y2="9" width="0.5" layer="1"/>
+<wire x1="4" y1="9" x2="5" y2="9" width="0.5" layer="1"/>
+<wire x1="5" y1="9" x2="5.31" y2="9.31" width="0.5" layer="1"/>
+<wire x1="5.31" y1="9.31" x2="5.31" y2="13.69" width="0.5" layer="1"/>
 </signal>
 <signal name="V+">
 <contactref element="U$1" pad="1"/>
 <contactref element="JP1" pad="3"/>
-<wire x1="16.5424" y1="6.3824" x2="16.58" y2="6.42" width="0.4064" layer="1"/>
-<wire x1="16.58" y1="6.42" x2="21.59" y2="11.43" width="0.4064" layer="1"/>
-<wire x1="16.58" y1="6.42" x2="7.5926375" y2="6.42" width="0.4064" layer="1"/>
-<wire x1="7.5926375" y1="6.42" x2="7.5550375" y2="6.3824" width="0.4064" layer="1"/>
-<wire x1="5.69668125" y1="6.9824" x2="5.1276" y2="6.9824" width="0.4064" layer="1"/>
-<wire x1="5.1276" y1="6.9824" x2="5.08" y2="7.03" width="0.4064" layer="1"/>
-<wire x1="7.5550375" y1="6.3824" x2="6.29668125" y2="6.3824" width="0.4064" layer="1"/>
-<wire x1="6.29668125" y1="6.3824" x2="5.69668125" y2="6.9824" width="0.4064" layer="1"/>
+<wire x1="5.1276" y1="6.9824" x2="5.08" y2="6.98" width="0.4064" layer="1"/>
+<wire x1="5.08" y1="6.98" x2="5.85591875" y2="6.98" width="0.5" layer="1"/>
+<wire x1="5.85591875" y1="6.98" x2="6.58331875" y2="6.2526" width="0.5" layer="1"/>
+<wire x1="6.58331875" y1="6.2526" x2="16.4126" y2="6.2526" width="0.5" layer="1"/>
+<wire x1="16.4126" y1="6.2526" x2="21.59" y2="11.43" width="0.5" layer="1"/>
 </signal>
 <signal name="V0">
 <contactref element="U$1" pad="4"/>
 <contactref element="JP1" pad="2"/>
-<wire x1="7.28" y1="5.73" x2="18.43" y2="5.73" width="0.4064" layer="1"/>
-<wire x1="18.43" y1="5.73" x2="21.59" y2="8.89" width="0.4064" layer="1"/>
+<wire x1="21.59" y1="8.89" x2="20.89" y2="8.89" width="0.5" layer="1"/>
+<wire x1="20.89" y1="8.89" x2="17" y2="5" width="0.5" layer="1"/>
+<wire x1="17" y1="5" x2="7.36" y2="5" width="0.5" layer="1"/>
+<wire x1="7.36" y1="5" x2="7.28" y2="5.08" width="0.5" layer="1"/>
 </signal>
 <signal name="V-">
 <contactref element="U$1" pad="3"/>
 <contactref element="JP1" pad="1"/>
-<wire x1="5.08" y1="5.73" x2="5.81" y2="5" width="0.4064" layer="1"/>
-<wire x1="20.24" y1="5" x2="21.59" y2="6.35" width="0.4064" layer="1"/>
-<wire x1="5.81" y1="5" x2="20.24" y2="5" width="0.4064" layer="1"/>
+<wire x1="21.59" y1="6.35" x2="19.24" y2="4" width="0.5" layer="1"/>
+<wire x1="5" y1="4" x2="5" y2="5" width="0.5" layer="1"/>
+<wire x1="5" y1="5" x2="5.08" y2="5.08" width="0.5" layer="1"/>
+<wire x1="19.24" y1="4" x2="5" y2="4" width="0.5" layer="1"/>
 </signal>
 </signals>
