File: particle_detector/Breakout/Comparator Breakout MCP6541.brd (EAGLE design)
At the start: 23 x 18 mm, 3 parts

Commit message: revised boards from a while ago
Changed lines of the file:
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@@
 <wire x1="7.3" y1="13.78" x2="7.49" y2="13.97" width="0.5" layer="1"/>
 <wire x1="7.49" y1="13.97" x2="21.59" y2="13.97" width="0.4064" layer="1"/>
-<wire x1="7.2" y1="6.95" x2="7.2" y2="13.68" width="0.4064" layer="1"/>
+<wire x1="7.2" y1="6.9" x2="7.2" y2="13.68" width="0.4064" layer="1"/>
 <wire x1="7.2" y1="13.68" x2="7.3" y2="13.78" width="0.5" layer="1"/>
 </signal>
@@
 <wire x1="6.2476" y1="14.69668125" x2="8.06091875" y2="16.51" width="0.4064" layer="1"/>
 <wire x1="8.06091875" y1="16.51" x2="21.59" y2="16.51" width="0.4064" layer="1"/>
-<wire x1="4.43091875" y1="6.3" x2="3.266" y2="7.46491875" width="0.4064" layer="1"/>
-<wire x1="3.266" y1="7.46491875" x2="3.266" y2="8" width="0.4064" layer="1"/>
-<wire x1="5" y1="6.3" x2="4.43091875" y2="6.3" width="0.4064" layer="1"/>
-<wire x1="3.266" y1="8" x2="5.4" y2="10.134" width="0.4064" layer="1"/>
-<wire x1="5.4" y1="10.134" x2="5.4" y2="13.78" width="0.4064" layer="1"/>
+<wire x1="5.4" y1="13.78" x2="5.4" y2="9.4" width="0.5" layer="1"/>
+<wire x1="5.4" y1="9.4" x2="3.266" y2="7.266" width="0.5" layer="1"/>
+<wire x1="3.266" y1="7.266" x2="3.266" y2="7" width="0.5" layer="1"/>
+<wire x1="3.266" y1="7" x2="4.316" y2="5.95" width="0.5" layer="1"/>
+<wire x1="4.316" y1="5.95" x2="5" y2="5.95" width="0.5" layer="1"/>
 </signal>
 <signal name="V+">
 <contactref element="U$1" pad="3"/>
 <contactref element="JP1" pad="1"/>
-<wire x1="5" y1="5.65" x2="5.65" y2="5" width="0.4064" layer="1"/>
-<wire x1="20.24" y1="5" x2="21.59" y2="6.35" width="0.4064" layer="1"/>
-<wire x1="5.65" y1="5" x2="20.24" y2="5" width="0.4064" layer="1"/>
+<wire x1="5.77591875" y1="5" x2="5" y2="5" width="0.5" layer="1"/>
+<wire x1="6.50331875" y1="4.2726" x2="5.77591875" y2="5" width="0.5" layer="1"/>
+<wire x1="19.5126" y1="4.2726" x2="6.50331875" y2="4.2726" width="0.5" layer="1"/>
+<wire x1="21.59" y1="6.35" x2="19.5126" y2="4.2726" width="0.5" layer="1"/>
 </signal>
 <signal name="V0">
 <contactref element="U$1" pad="1"/>
 <contactref element="JP1" pad="3"/>
-<wire x1="5" y1="6.95" x2="5.95" y2="6.95" width="0.4064" layer="1"/>
-<wire x1="5.95" y1="6.95" x2="6" y2="7" width="0.4064" layer="1"/>
-<wire x1="6" y1="7" x2="6.3476" y2="6.6524" width="0.4064" layer="1"/>
-<wire x1="6.3476" y1="6.6524" x2="6.3476" y2="6.58331875" width="0.4064" layer="1"/>
-<wire x1="6.3476" y1="6.58331875" x2="6.67851875" y2="6.2524" width="0.4064" layer="1"/>
-<wire x1="14.43" y1="11.43" x2="21.59" y2="11.43" width="0.4064" layer="1"/>
-<wire x1="6.67851875" y1="6.2524" x2="9.2524" y2="6.2524" width="0.4064" layer="1"/>
-<wire x1="9.2524" y1="6.2524" x2="14.43" y2="11.43" width="0.4064" layer="1"/>
+<wire x1="21.59" y1="11.43" x2="15.43" y2="11.43" width="0.5" layer="1"/>
+<wire x1="15.43" y1="11.43" x2="10" y2="6" width="0.5" layer="1"/>
+<wire x1="5.69668125" y1="6.6774" x2="5.2226" y2="6.6774" width="0.5" layer="1"/>
+<wire x1="5.2226" y1="6.6774" x2="5" y2="6.9" width="0.5" layer="1"/>
+<wire x1="10" y1="6" x2="6.37408125" y2="6" width="0.5" layer="1"/>
+<wire x1="6.37408125" y1="6" x2="5.69668125" y2="6.6774" width="0.5" layer="1"/>
 </signal>
 <signal name="V-">
 <contactref element="U$1" pad="4"/>
 <contactref element="JP1" pad="2"/>
-<wire x1="7.2" y1="5.65" x2="18.35" y2="5.65" width="0.4064" layer="1"/>
-<wire x1="18.35" y1="5.65" x2="21.59" y2="8.89" width="0.4064" layer="1"/>
+<wire x1="7.2" y1="5" x2="14" y2="5" width="0.5" layer="1"/>
+<wire x1="14" y1="5" x2="17.89" y2="8.89" width="0.5" layer="1"/>
+<wire x1="17.89" y1="8.89" x2="21.59" y2="8.89" width="0.5" layer="1"/>
 </signal>
 </signals>
